File: USB-Serial_HighSpeed.kicad_pcb (KiCad board)
At the start: 2 copper layers, 35.5 x 16.5 mm, 48 parts, among them J1 USB_C_Receptacle_USB2.0, J2 Conn_01x04, SW1 SW_DPDT_x2, U1 FT232H, U2 SP3485CN, U3 93LCxxBxxOT, Y1 12MHz

Commit message: GND調整
Connections:
- J1 pad S1: Net-(J1-PadS1) -> GND
Routing:
- net GND: track 146.9 -> 163.7 mm, vias 13 -> 22

Commit message: これで出す
Parts:
- removed C17, C18: 12p, Capacitor_SMD:C_0402_1005Metric
- R17, R7, R8: value R -> 1k
- R18: value R -> 120
- Y1: value 12MHz -> Crystal_GND2_Small; footprint Crystal_my:NDK_Crystal_SMD_3225_2Pads -> Crystal:Resonator_SMD_muRata_CSTxExxV-3Pin_3.0x1.1mm
- moved R18 4.88 mm to (189.3, 113.9), turned to 0 degrees
- moved SW1 1.40 mm to (193.0, 109.5)
- moved Y1 0.32 mm to (176.4, 104.0), turned to 180 degrees
Connections:
- R18 pad 1: Net-(J2-Pad3) -> Net-(J2-Pad4)
- SW1 pad 2: Net-(R18-Pad2) -> Net-(J2-Pad3)
- SW1 pad 3: Net-(J2-Pad4) -> Net-(R18-Pad2)
- U1 pad 1: Net-(C17-Pad1) -> Net-(U1-Pad1)
- U1 pad 2: Net-(C18-Pad1) -> Net-(U1-Pad2)
- Y1 pad 1: Net-(C18-Pad1) -> Net-(U1-Pad1)
- Y1 pad 2: Net-(C17-Pad1) -> GND
Routing:
- net +3V3: track 73.5 -> 85.2 mm
- net Net-(F1-Pad2): track 10.9 -> 20.6 mm
- net Net-(C18-Pad1): track 6.67 -> 0.00 mm
- net Net-(C17-Pad1): track 4.93 -> 0.00 mm
- net Net-(U1-Pad2): track 0.00 -> 4.08 mm
- net Net-(U1-Pad1): track 0.00 -> 2.42 mm
- net /TXD: track 11.5 -> 10.2 mm
- net Net-(R18-Pad2): track 1.80 -> 2.89 mm
- net Net-(J2-Pad4): track 20.5 -> 19.6 mm
- net /TXDEN: track 6.01 -> 5.28 mm
