File: USB-Serial_HighSpeed.sch (KiCad schematic (older format))
At the start: 30 parts

Commit message: できた
Parts:
- removed Y?: Crystal_GND2, symbol Device:Crystal_GND2
- added C14, C15: 0.1u, Capacitor_SMD:C_0402_1005Metric, symbol Device:C
- added C16: 10n, Capacitor_SMD:C_0402_1005Metric, symbol Device:C
- added C17, C18: 12p, Capacitor_SMD:C_0402_1005Metric, symbol Device:C
- added D3: LED, LED_SMD:LED_0603_1608Metric, symbol Device:LED
- added J2: Conn_01x04, Connector_PinHeader_2.54mm:PinHeader_1x04_P2.54mm_Horizontal, symbol Connector_Generic:Conn_01x04
- added R10: 2k, Resistor_SMD:R_0402_1005Metric, symbol Device:R
- added R11, R12, R9: 10k, Resistor_SMD:R_0402_1005Metric, symbol Device:R
- added R15, R16: 0, Resistor_SMD:R_0402_1005Metric, symbol Device:R
- added R17: R, Resistor_SMD:R_0402_1005Metric, symbol Device:R
- added R18: R, Resistor_SMD:R_0603_1608Metric, symbol Device:R
- added SW1: SW_DPDT_x2, Button_Switch_SMD:SW_SPDT_PCM12, symbol Switch:SW_DPDT_x2
- added U2: SP3485CN, Package_SO:SOIC-8_3.9x4.9mm_P1.27mm, symbol Interface_UART:SP3485CN
- added U3: 93LCxxBxxOT, Package_TO_SOT_SMD:SOT-23-6, symbol Memory_EEPROM:93LCxxBxxOT
- added Y1: 12MHz, Crystal_my:NDK_Crystal_SMD_3225_2Pads, symbol Device:Crystal
- C1, C10, C2, C9: renamed from C?; footprint (none) -> Capacitor_SMD:C_0603_1608Metric
- C11, C12, C13, C3, C4, C5, C6, C7, C8: renamed from C?; footprint (none) -> Capacitor_SMD:C_0402_1005Metric
- D1, D2: renamed from D?; footprint (none) -> LED_SMD:LED_0603_1608Metric
- F1: renamed from F?; footprint (none) -> Fuse:Fuse_0603_1608Metric
- J1: renamed from J?; footprint (none) -> Connector_USB:USB_C_Receptacle_GCT_USB4085
- L1, L2, L3: renamed from L?; footprint (none) -> Inductor_SMD:L_0603_1608Metric
- R1, R2, R3, R4, R5, R6, R7, R8: renamed from R?; footprint (none) -> Resistor_SMD:R_0402_1005Metric
- U1: renamed from U?; footprint (none) -> Package_QFP:LQFP-48_7x7mm_P0.5mm
Connections:
- net +3V3: now also C11.1, C12.1, C13.1, R7.1, R8.1, U1.12 (VCCIO), U1.24 (VCCIO), U1.46 (VCCIO), C15.1, R11.2, R12.2, R9.2, U3.6 (VCC); no longer D1.2 (A), D2.2 (A)
- net GND: now also C14.2, C15.2, C16.2, C17.2, C18.2, D3.1 (K), J2.1 (Pin_1), U2.5 (GND), U3.2 (GND)
- net RXD: now also R15.2, U2.1 (RO)
- net RXLED: now also D2.1 (K); no longer R8.2
- net TXD: now also R16.2, U2.4 (DI)
- net TXDEN: now also U2.2 (~RE~), U2.3 (DE)
- net TXLED: now also D1.1 (K); no longer R7.2
- net at F1.1, J1.A4 (VBUS), J1.A9 (VBUS)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: now also C16.1
- net at U1.1 (XCSI): now also C17.1, Y1.2
- net at U1.2 (XCSO): now also C18.1, Y1.1
- net +5V: now reaches C2.1, C5.1, L1.2, U1.40 (VREGIN)
- net +5V: now also C14.1, J2.2 (Pin_2), U2.8 (VCC)
- net EEDATA: now reaches U1.43 (EEDATA)
- net EEDATA: now also R10.1, R12.1, U3.3 (DI)
- net EECLK: now reaches U1.44 (EECLK)
- net EECLK: now also R11.1, U3.4 (CLK)
- net EECS: now reaches U1.45 (EECS)
- net EECS: now also R9.1, U3.5 (CS)
- net at F1.2, L1.1: now also R17.1
- new net: D1.2 (A), R7.2
- new net: D2.2 (A), R8.2
- new net: J2.3 (Pin_3), R16.1, R18.1, U2.6 (A)
- new net: J2.4 (Pin_4), R15.1, SW1.3 (C), U2.7 (B)
- new net: R10.2, U3.1 (DO)
- new net: D3.2 (A), R17.2
- new net: R18.2, SW1.2 (B)
- no-connect marks 18 -> 16
Other:
- moved on the sheet: C1, C10, C11, C12, C13, C2, C3, C4, C5, C6, C7, C8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

Commit message: これで出す
Parts:
- removed C17, C18: 12p, Capacitor_SMD:C_0402_1005Metric, symbol Device:C
- removed Y1: 12MHz, Crystal_my:NDK_Crystal_SMD_3225_2Pads, symbol Device:Crystal
- added Y1: Crystal_GND2_Small, Crystal:Resonator_SMD_muRata_CSTxExxV-3Pin_3.0x1.1mm, symbol Device:Crystal_GND2_Small
- R17, R7, R8: value R -> 1k
- R18: value R -> 120
Connections:
- net GND: now also J1.S1 (SHIELD), Y1.2
- net at U1.1 (XCSI): now also Y1.1
- net at U1.2 (XCSO): now also Y1.3
- net at J2.3 (Pin_3), R16.1, U2.6 (A): now also SW1.2 (B); no longer R18.1
- net at J2.4 (Pin_4), R15.1, U2.7 (B): now also R18.1; no longer SW1.3 (C)
- net at R18.2: now also SW1.3 (C); no longer SW1.2 (B)
Other:
- moved on the sheet: R18
Changed lines of the file:
@@
 P 7950 1400
 F 0 "R7" H 8020 1446 50  0000 L CNN
-F 1 "R" H 8020 1355 50  0000 L CNN
+F 1 "1k" H 8020 1355 50  0000 L CNN
 F 2 "Resistor_SMD:R_0402_1005Metric" V 7880 1400 50  0001 C CNN
 F 3 "~" H 7950 1400 50  0001 C CNN
@@
 P 8300 1400
 F 0 "R8" H 8370 1446 50  0000 L CNN
-F 1 "R" H 8370 1355 50  0000 L CNN
+F 1 "1k" H 8370 1355 50  0000 L CNN
 F 2 "Resistor_SMD:R_0402_1005Metric" V 8230 1400 50  0001 C CNN
 F 3 "~" H 8300 1400 50  0001 C CNN
@@
 $EndComp
 $Comp
-L Device:Crystal Y1
-U 1 1 5F409A27
-P 4350 5150
-F 0 "Y1" V 4396 5019 50  0000 R CNN
-F 1 "12MHz" V 4305 5019 50  0000 R CNN
-F 2 "Crystal_my:NDK_Crystal_SMD_3225_2Pads" H 4350 5150 50  0001 C CNN
-F 3 "~" H 4350 5150 50  0001 C CNN
-	1    4350 5150
-	0    -1   -1   0
-$EndComp
-$Comp
-L Device:C C18
-U 1 1 5F415253
-P 4350 5600
-F 0 "C18" H 4465 5646 50  0000 L CNN
-F 1 "12p" H 4465 5555 50  0000 L CNN
-F 2 "Capacitor_SMD:C_0402_1005Metric" H 4388 5450 50  0001 C CNN
-F 3 "~" H 4350 5600 50  0001 C CNN
-	1    4350 5600
-	1    0    0    -1
-$EndComp
-Wire Wire Line
-	4350 5350 4350 5450
-Wire Wire Line
-	4350 5350 4350 5300
-Connection ~ 4350 5350
-Wire Wire Line
-	4350 5350 5150 5350
-Wire Wire Line
-	5150 4950 4350 4950
-Wire Wire Line
-	4350 4950 4350 5000
-$Comp
-L Device:C C17
-U 1 1 5F424F9D
-P 3850 5600
-F 0 "C17" H 3965 5646 50  0000 L CNN
-F 1 "12p" H 3965 5555 50  0000 L CNN
-F 2 "Capacitor_SMD:C_0402_1005Metric" H 3888 5450 50  0001 C CNN
-F 3 "~" H 3850 5600 50  0001 C CNN
-	1    3850 5600
-	1    0    0    -1
-$EndComp
-Wire Wire Line
-	3850 5450 3850 4950
-Wire Wire Line
-	3850 4950 4350 4950
-Connection ~ 4350 4950
-$Comp
-L power:GND #PWR0135
-U 1 1 5F42ABAB
-P 4350 5850
-F 0 "#PWR0135" H 4350 5600 50  0001 C CNN
-F 1 "GND" H 4355 5677 50  0000 C CNN
-F 2 "" H 4350 5850 50  0001 C CNN
-F 3 "" H 4350 5850 50  0001 C CNN
-	1    4350 5850
-	1    0    0    -1
-$EndComp
-Wire Wire Line
-	4350 5850 4350 5800
-Wire Wire Line
-	4350 5800 3850 5800
-Wire Wire Line
-	3850 5800 3850 5750
-Connection ~ 4350 5800
-Wire Wire Line
-	4350 5800 4350 5750
-$Comp
 L Memory_EEPROM:93LCxxBxxOT U3
 U 1 1 5F438946
@@
 P 3100 2950
 F 0 "R17" H 3170 2996 50  0000 L CNN
-F 1 "R" H 3170 2905 50  0000 L CNN
+F 1 "1k" H 3170 2905 50  0000 L CNN
 F 2 "Resistor_SMD:R_0402_1005Metric" V 3030 2950 50  0001 C CNN
 F 3 "~" H 3100 2950 50  0001 C CNN
@@
 L Device:R R18
 U 1 1 5F8A61BA
-P 10300 4500
-F 0 "R18" H 10370 4546 50  0000 L CNN
-F 1 "R" H 10370 4455 50  0000 L CNN
-F 2 "Resistor_SMD:R_0603_1608Metric" V 10230 4500 50  0001 C CNN
-F 3 "~" H 10300 4500 50  0001 C CNN
-	1    10300 4500
-	1    0    0    -1
-$EndComp
-Wire Wire Line
-	10300 4650 10300 4700
+P 10200 4500
+F 0 "R18" H 10270 4546 50  0000 L CNN
+F 1 "120" H 10270 4455 50  0000 L CNN
+F 2 "Resistor_SMD:R_0603_1608Metric" V 10130 4500 50  0001 C CNN
+F 3 "~" H 10200 4500 50  0001 C CNN
+	1    10200 4500
+	1    0    0    -1
+$EndComp
 Wire Wire Line
 	10200 5100 10200 5150
 Wire Wire Line
 	10200 4100 10650 4100
-Wire Wire Line
-	10300 4350 10300 4000
 Connection ~ 10300 4000
 Wire Wire Line
@@
 	10100 4700 10200 4700
 Wire Wire Line
-	10200 4700 10200 4200
+	10200 4700 10200 4650
 Wire Wire Line
 	10100 5150 10200 5150
@@
 	3650 2650 3650 3250
 Connection ~ 3650 3250
+$Comp
+L power:GND #PWR0138
+U 1 1 5FA707BB
+P 1900 5350
+F 0 "#PWR0138" H 1900 5100 50  0001 C CNN
+F 1 "GND" H 1905 5177 50  0000 C CNN
+F 2 "" H 1900 5350 50  0001 C CNN
+F 3 "" H 1900 5350 50  0001 C CNN
+	1    1900 5350
+	1    0    0    -1
+$EndComp
+$Comp
+L Device:Crystal_GND2_Small Y1
+U 1 1 5FA8EC03
+P 4350 5150
+F 0 "Y1" V 4304 5238 50  0000 L CNN
+F 1 "Crystal_GND2_Small" V 4395 5238 50  0000 L CNN
+F 2 "Crystal:Resonator_SMD_muRata_CSTxExxV-3Pin_3.0x1.1mm" H 4350 5150 50  0001 C CNN
+F 3 "~" H 4350 5150 50  0001 C CNN
+	1    4350 5150
+	0    1    1    0
+$EndComp
+Wire Wire Line
+	5150 4950 4350 4950
+Wire Wire Line
+	4350 4950 4350 5050
+Wire Wire Line
+	5150 5350 4350 5350
+Wire Wire Line
+	4350 5350 4350 5250
+$Comp
+L power:GND #PWR0135
+U 1 1 5FAA3BAA
+P 4100 5200
+F 0 "#PWR0135" H 4100 4950 50  0001 C CNN
+F 1 "GND" H 4105 5027 50  0000 C CNN
+F 2 "" H 4100 5200 50  0001 C CNN
+F 3 "" H 4100 5200 50  0001 C CNN
+	1    4100 5200
+	1    0    0    -1
+$EndComp
+Wire Wire Line
+	4250 5150 4100 5150
+Wire Wire Line
+	4100 5150 4100 5200
+Wire Wire Line
+	10200 4350 10200 4200
+Wire Wire Line
+	10300 4000 10300 4700
 $EndSCHEMATC
